File: 04 Electrical/Interconnect PCB V1.1 - footprint adjusted/Interconnect PCB.kicad_pcb (KiCad board)
At the start: 2 copper layers, 96 x 75 mm, 12 parts, among them J1 MSTB-2,5-2-G, T1 ButtonUp, T2 ButtonSelect, T3 ButtonDown, U1 mini_esp32, U2 ILI9341_touch, U3 OpenTherm_Master_Shield, U4 DS18B20, U5 DS18B20, U6 DS18B20, U7 DS18B20

Commit message: PCB modifications
Parts:
- moved J1 7.37 mm to (166.1, 121.0)
Routing:
- net Net-(J1-Pad1): track 7.57 -> 12.2 mm
- net Net-(J1-Pad2): track 17.2 -> 21.7 mm
Other:
- board text added: "ROOMTHERMOSTAT V1.1"
- board text added: "https://github.com/henkjannl/RoomThermostat"
- board text added: "unconnected"
