File: 04 Electrical/Opentherm interface/Simulations/Test 07. Component assignment/Test 07. Component assignment.kicad_sch (KiCad schematic)
At the start: 21 parts, among them J1 OpenTherm, J2 Controller, Q1 MMBT2907A, U1 EL357N-G, U2 EL357N-G

Commit message: mch
Parts:
- C1, C3: LCSC Part # (none) -> C57112
- C2, C4: LCSC Part # (none) -> C1604
- D1, D2, D3, D4: LCSC Part # (none) -> C2128
- D5: LCSC Part # (none) -> C5190168
- D6: LCSC Part # (none) -> C5299435
- D7: LCSC Part # (none) -> C726993
- J1, J2: now not fitted
- Q1: LCSC Part # (none) -> C916373
- R1: LCSC Part # (none) -> C17540
- R2: LCSC Part # (none) -> C17471
- R3, R5: LCSC Part # (none) -> C17630
- R4: LCSC Part # (none) -> C4310
- U1, U2: LCSC Part # (none) -> C29981
Changed lines of the file:
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@@
+			)
+		)
+		(property "LCSC Part #" "C17630"
+			(at 177.8 102.87 0)
+			(effects
+				(font
+					(size 1.27 1.27)
+				)
+				(hide yes)
 			)
 		)
@@
 			)
 		)
+		(property "LCSC Part #" "C726993"
+			(at 144.78 97.79 0)
+			(effects
+				(font
+					(size 1.27 1.27)
+				)
+				(hide yes)
+			)
+		)
 		(pin "1"
 		)
@@
 			)
 		)
+		(property "LCSC Part #" "C2128"
+			(at 82.55 80.01 0)
+			(effects
+				(font
+					(size 1.27 1.27)
+				)
+				(hide yes)
+			)
+		)
 		(pin "2"
 		)
@@
 			)
 		)
+		(property "LCSC Part #" "C1604"
+			(at 139.7 73.66 0)
+			(effects
+				(font
+					(size 1.27 1.27)
+				)
+				(hide yes)
+			)
+		)
 		(pin "1"
 		)
@@
 				)
 				(justify bottom)
+				(hide yes)
+			)
+		)
+		(property "LCSC Part #" "C29981"
+			(at 167.64 95.25 0)
+			(effects
+				(font
+					(size 1.27 1.27)
+				)
 				(hide yes)
 			)
@@
 		)
 		(property "Sim.Params" "m=0.33 is=1e-14 rs=0.5 n=1.06 tt=5n cjo=1e-12 vj=0.75 fc=0.5"
+			(at 82.55 59.69 0)
+			(effects
+				(font
+					(size 1.27 1.27)
+				)
+				(hide yes)
+			)
+		)
+		(property "LCSC Part #" "C2128"
 			(at 82.55 59.69 0)
 			(effects
@@
 			)
 		)
+		(property "LCSC Part #" "C5299435"
+			(at 129.54 97.79 0)
+			(effects
+				(font
+					(size 1.27 1.27)
+				)
+				(hide yes)
+			)
+		)
 		(pin "1"
 		)
@@
 		(in_bom yes)
 		(on_board yes)
-		(dnp no)
+		(dnp yes)
 		(fields_autoplaced yes)
 		(property "Reference" "J1"
@@
 			)
 		)
+		(property "LCSC Part #" "C4310"
+			(at 173.99 67.31 0)
+			(effects
+				(font
+					(size 1.27 1.27)
+				)
+				(hide yes)
+			)
+		)
 		(pin "2"
 		)
@@
 			)
 		)
+		(property "LCSC Part #" "C29981"
+			(at 153.67 69.85 0)
+			(effects
+				(font
+					(size 1.27 1.27)
+				)
+				(hide yes)
+			)
+		)
 		(pin "4"
 		)
@@
 			)
 		)
+		(property "LCSC Part #" "C57112"
+			(at 124.46 81.28 0)
+			(effects
+				(font
+					(size 1.27 1.27)
+				)
+				(hide yes)
+			)
+		)
 		(pin "1"
 		)
@@
 			)
 		)
+		(property "LCSC Part #" "C1604"
+			(at 167.64 72.39 0)
+			(effects
+				(font
+					(size 1.27 1.27)
+				)
+				(hide yes)
+			)
+		)
 		(pin "1"
 		)
@@
 			)
 		)
+		(property "LCSC Part #" "C17630"
+			(at 129.54 59.69 0)
+			(effects
+				(font
+					(size 1.27 1.27)
+				)
+				(hide yes)
+			)
+		)
 		(pin "2"
 		)
@@
 			)
 		)
+		(property "LCSC Part #" "C2128"
+			(at 82.55 64.77 0)
+			(effects
+				(font
+					(size 1.27 1.27)
+				)
+				(hide yes)
+			)
+		)
 		(pin "2"
 		)
@@
 		(in_bom yes)
 		(on_board yes)
-		(dnp no)
+		(dnp yes)
 		(fields_autoplaced yes)
 		(property "Reference" "J2"
@@
 			)
 		)
+		(property "LCSC Part #" "C2128"
+			(at 82.55 85.09 0)
+			(effects
+				(font
+					(size 1.27 1.27)
+				)
+				(hide yes)
+			)
+		)
 		(pin "2"
 		)
@@
 			)
 		)
+		(property "LCSC Part #" "C17540"
+			(at 113.03 82.55 0)
+			(effects
+				(font
+					(size 1.27 1.27)
+				)
+				(hide yes)
+			)
+		)
 		(pin "2"
 		)
@@
 			)
 		)
+		(property "LCSC Part #" "C57112"
+			(at 154.94 97.79 0)
+			(effects
+				(font
+					(size 1.27 1.27)
+				)
+				(hide yes)
+			)
+		)
 		(pin "1"
 		)
@@
 		)
 		(property "Sim.Params" "is=1.7E-14 bf=240 nf=1 vaf=100 ikf=0.2 ise=1E-13 ne=2 br=7 nr=1 var=10 ikr=0.03 isc=1E-13 nc=2 rb=10 re=0.5 rc=1 cje=13.5p vje=0.6 mje=0.33 tf=0.35n cjc=6.5p vjc=0.5 mjc=0.4 tr=30n xtb=1.5 eg=1.11 kf=0 af=1"
+			(at 115.57 67.31 0)
+			(effects
+				(font
+					(size 1.27 1.27)
+				)
+				(hide yes)
+			)
+		)
+		(property "LCSC Part #" "C916373"
 			(at 115.57 67.31 0)
 			(effects
@@
 			)
 		)
+		(property "LCSC Part #" "C5190168"
+			(at 102.87 97.79 0)
+			(effects
+				(font
+					(size 1.27 1.27)
+				)
+				(hide yes)
+			)
+		)
 		(pin "1"
 		)
@@
 			(at 113.03 97.79 0)
 			(effects
+				(font
+					(size 1.27 1.27)
+				)
+				(hide yes)
+			)
+		)
+		(property "LCSC Part #" "C17471"
+			(at 113.03 97.79 0)
+			(effects
