File: 04 Electrical/Opentherm interface/Simulations/Test 08. With ESP32 mini/Test 08. With ESP32 mini.kicad_sch (KiCad schematic)
At the start: 31 parts, among them J1 OpenTherm, J2 Laser range sensor, J3 ST7789, J4 Encoder, J5 Encoder, Q1 MMBT2907A, SW1 RotaryEncoder_Switch, U1 DS18S20, U2 DS18S20, U3 DS18S20, U4 DS18S20, U5 EL357N-G, U6 EL357N-G, U7 mini_esp32

Commit message: mch
Parts:
- C1, C3: LCSC Part #  (none) -> C57112
- C2, C4: LCSC Part #  (none) -> C1604
- D1, D2, D3, D4: LCSC Part #  (none) -> C2128
- D5: LCSC Part #  (none) -> C5190168
- D6: LCSC Part #  (none) -> C5299435
- D7: LCSC Part #  (none) -> C726993
- J1, J2, J3, J4, U7: now not fitted
- Q1: LCSC Part #  (none) -> C916373
- R1: LCSC Part #  (none) -> C25292
- R2: LCSC Part #  (none) -> C17471
- R3, R6: LCSC Part #  (none) -> C17630
- R4: LCSC Part #  (none) -> C23162
- R5: LCSC Part #  (none) -> C4310
- U3: now left out of the parts list
- U5, U6: LCSC Part #  (none) -> C29981
Other:
- moved on the sheet: U1, U2
