File: 04 Electrical/Opentherm interface/PCB design/Test 09. With ESP module/Thermometers.kicad_sch (KiCad schematic)
At the start: 5 parts, among them U6 DS18S20, U7 DS18S20, U8 DS18S20, U9 DS18S20

Commit message: Component assignment
Parts:
- R10: footprint Resistor_SMD:R_0201_0603Metric -> Resistor_SMD:R_0603_1608Metric
Changed lines of the file:
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@@
 			)
 		)
-		(property "Footprint" "Resistor_SMD:R_0201_0603Metric"
+		(property "Footprint" "Resistor_SMD:R_0603_1608Metric"
 			(at 197.358 86.36 90)
 			(effects
