File: 04 Electrical/Redesign PCB 3.0/PCB design/Test 09. With ESP module/LEDs.kicad_sch (KiCad schematic)
At the start: 8 parts, among them Q2 LBSS138LT1G-ES

Commit message: Routing PCB test 9
Parts:
- removed C13: 10u, Capacitor_SMD:C_0402_1005Metric, symbol Device:C
- removed D18, D19, D20: WS2812B-2020, LED_SMD:LED_WS2812B_PLCC4_5.0x5.0mm_P3.2mm, symbol LED:WS2812B
- removed Q2: LBSS138LT1G-ES, Package_TO_SOT_SMD:SOT-23, symbol Transistor_FET:BSS138
- removed R11, R12, R13: 10k, Resistor_SMD:R_0603_1608Metric, symbol Device:R
Connections:
- no-connect marks 1 -> 0
