File: 04 Electrical/Redesign PCB 3.0/PCB design/Test 09. With ESP module/Test 09. With ESP module.kicad_sch (KiCad schematic)
At the start: 0 parts

Commit message: As ordered at JLCPCB
Other:
- removed sheet LEDs
Changed lines of the file:
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@@
 	(polyline
 		(pts
-			(xy 180.34 114.3) (xy 180.34 105.41)
-		)
-		(stroke
-			(width 0)
-			(type default)
-		)
-	)
-	(polyline
-		(pts
-			(xy 198.12 88.9) (xy 203.2 88.9)
-		)
-		(stroke
-			(width 0)
-			(type default)
-		)
-	)
-	(polyline
-		(pts
-			(xy 139.7 114.3) (xy 139.7 105.41)
-		)
-		(stroke
-			(width 0)
-			(type default)
-		)
-	)
-	(polyline
-		(pts
-			(xy 96.52 114.3) (xy 96.52 105.41)
+			(xy 203.2 88.9) (xy 198.12 88.9)
+		)
+		(stroke
+			(width 0)
+			(type default)
+		)
+	)
+	(polyline
+		(pts
+			(xy 171.45 114.3) (xy 171.45 105.41)
+		)
+		(stroke
+			(width 0)
+			(type default)
+		)
+	)
+	(polyline
+		(pts
+			(xy 106.68 114.3) (xy 106.68 105.41)
 		)
 		(stroke
@@
 	)
 	(sheet
-		(at 123.19 114.3)
-		(size 33.02 30.48)
+		(at 144.78 114.3)
+		(size 53.34 30.48)
 		(fields_autoplaced yes)
 		(stroke
@@
 		)
 		(property "Sheetname" "Display"
-			(at 123.19 113.5884 0)
+			(at 144.78 113.5884 0)
 			(effects
 				(font
@@
 		)
 		(property "Sheetfile" "Display.kicad_sch"
-			(at 123.19 145.3646 0)
+			(at 144.78 145.3646 0)
 			(effects
 				(font
@@
 	(sheet
 		(at 80.01 114.3)
-		(size 33.02 30.48)
+		(size 53.34 30.48)
 		(fields_autoplaced yes)
 		(stroke
@@
 			(project "Test 09. With ESP module"
 				(path "/dee7d3c3-6abb-4cb3-8df4-3e3e37989a04"
-					(page "9")
+					(page "8")
 				)
 			)
@@
 	)
 	(sheet
-		(at 162.56 114.3)
-		(size 35.56 30.48)
+		(at 203.2 74.93)
+		(size 30.48 30.48)
 		(fields_autoplaced yes)
 		(stroke
@@
 		)
 		(property "Sheetname" "Buttons"
-			(at 162.56 113.5884 0)
+			(at 203.2 74.2184 0)
 			(effects
 				(font
@@
 		)
 		(property "Sheetfile" "Buttons.kicad_sch"
-			(at 162.56 145.3646 0)
+			(at 203.2 105.9946 0)
 			(effects
 				(font
@@
 				)
 			)
-		)
-	)
-	(sheet
-		(at 203.2 71.12)
-		(size 30.48 34.29)
-		(fields_autoplaced yes)
-		(stroke
-			(width 0.1524)
-			(type solid)
-		)
-		(fill
-			(color 0 0 0 0.0000)
-		)
-		(property "Sheetname" "LEDs"
-			(at 203.2 70.4084 0)
-			(effects
-				(font
-					(size 1.27 1.27)
-				)
-				(justify left bottom)
-			)
-		)
-		(property "Sheetfile" "LEDs.kicad_sch"
-			(at 203.2 105.9946 0)
-			(effects
-				(font
-					(size 1.27 1.27)
-				)
-				(justify left top)
-			)
-		)
-		(instances
-			(project "Test 09. With ESP module"
-				(path "/dee7d3c3-6abb-4cb3-8df4-3e3e37989a04"
-					(page "8")
-				)
-			)
