File: 04 Electrical/Redesign PCB 3.0/PCB design/Test 09. With ESP module/Time_of_flight.kicad_sch (KiCad schematic)
At the start: 4 parts, among them U10 LP5907MFX-2.8/NOPB, U11 VL53L0CXV0DH/1

Commit message: Routing PCB test 9
Parts:
- removed C14: 0.1u, Capacitor_SMD:C_0603_1608Metric, symbol Device:C
- removed C15: 4.7pF, Capacitor_SMD:C_0603_1608Metric, symbol Device:C
- removed U10: LP5907MFX-2.8/NOPB, Package_TO_SOT_SMD:SOT-23-5, symbol Regulator_Linear:LP5907MFX-2.8
- removed U11: VL53L0CXV0DH/1, Sensor_Distance:ST_VL53L1x, symbol Sensor_Distance:VL53L0CXV0DH1
- added J4: VL6180, Connector_PinHeader_2.00mm:PinHeader_1x06_P2.00mm_Vertical, symbol Connector:Conn_01x06_Pin
Connections:
- net GND: now also J4.5 (Pin_5)
- net TOF_GPIO01: now also J4.2 (Pin_2)
- net TOF_SCL: now also J4.3 (Pin_3)
- net TOF_SDA: now also J4.4 (Pin_4)
- net TOF_XSHUT: now also J4.1 (Pin_1)
- net VCC_3V3: now also J4.6 (Pin_6)

Commit message: As ordered at JLCPCB
Parts:
- J3: renamed from J4; now not fitted
Changed lines of the file:
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@@
 		(in_bom yes)
 		(on_board yes)
-		(dnp no)
+		(dnp yes)
 		(fields_autoplaced yes)
-		(property "Reference" "J4"
+		(property "Reference" "J3"
 			(at 156.21 88.8999 0)
 			(effects
@@
 			)
 		)
+		(property "Comment" ""
+			(at 154.94 88.9 0)
+			(effects
+				(font
+					(size 1.27 1.27)
+				)
+				(hide yes)
+			)
+		)
 		(pin "2"
 		)
@@
 			(project ""
 				(path "/dee7d3c3-6abb-4cb3-8df4-3e3e37989a04/9496b48a-90bf-416c-bf1c-039c65c989b9"
-					(reference "J4")
+					(reference "J3")
 					(unit 1)
 				)
@@
 		(dnp no)
 		(fields_autoplaced yes)
-		(property "Reference" "#PWR036"
+		(property "Reference" "#PWR034"
 			(at 134.62 101.6 0)
 			(effects
@@
 			(project "Test 09. With ESP module"
 				(path "/dee7d3c3-6abb-4cb3-8df4-3e3e37989a04/9496b48a-90bf-416c-bf1c-039c65c989b9"
-					(reference "#PWR036")
+					(reference "#PWR034")
 					(unit 1)
 				)
