File: 04 Electrical/Redesign PCB 3.0/PCB design/Test 06. Simplified interface/Test 06. Simplified interface.kicad_sch (KiCad schematic)
At the start: 21 parts, among them Q1 MMBT5401, U1 NPN

Commit message: As ordered at JLCPCB
Parts:
- removed C1, C2: 2n2, symbol Device:C
- removed C3: 10n, symbol Device:C
- R1: value 200 -> 180
- R2: value 150 -> 100
Other:
- moved on the sheet: R4, U2, V1
